File: keyboard.kicad_pcb (KiCad board)
At the start: 2 copper layers, 454 x 125.4 mm, 238 parts, among them U1 STM32F072-LQFP48, U3 AMS1117-3.3, U4 USBLC6-2SC6

Commit message: power supply completion
Routing:
- net D-: track 64.3 -> 113.9 mm
- net 3.3V: track 111.1 -> 134.1 mm
- net Net-(R2-Pad2): track 0.00 -> 8.09 mm, vias 0 -> 2
- net Net-(R3-Pad2): track 0.00 -> 6.97 mm, vias 0 -> 2
- net D+: track 112.8 -> 105.8 mm
- net GND: track 0.00 -> 6.19 mm, vias 0 -> 2
- net VUSB: track 25.8 -> 29.5 mm, vias 0 -> 1
- added copper zone on B.Cu, net GND
- added copper zone on F.Cu, net VUSB
